Commit message: 0705 update

File: robots/allegro_hand_right.urdf (robot description, URDF)
Before this commit: robot allegro_hand_right, 21 links, 20 joints
Links:
- removed link link_0.0
- removed link link_1.0
- removed link link_10.0
- removed link link_11.0
- removed link link_11.0_tip
- removed link link_12.0
- removed link link_13.0
- removed link link_14.0
- removed link link_15.0
- removed link link_15.0_tip
- removed link link_2.0
- removed link link_3.0
- removed link link_3.0_tip
- removed link link_4.0
- removed link link_5.0
- removed link link_6.0
- removed link link_7.0
- removed link link_7.0_tip
- removed link link_8.0
- removed link link_9.0
- added link index_tip_tactile; collision mesh filename=./fingertip_V2_fixed2.STL scale=0.001 0.001 0.001
- added link link_0; collision mesh filename=./link_0.0.STL
- added link link_1; collision mesh filename=./link_1.0.STL
- added link link_10; collision mesh filename=./link_2.0.STL
- added link link_11; collision mesh filename=./link_3.0.STL
- added link link_12; collision mesh filename=./link_12.0_right.STL
- added link link_13; collision mesh filename=./link_13.0.STL
- added link link_14; collision mesh filename=./link_14.0.STL
- added link link_15; collision mesh filename=./link_15.0.STL
- added link link_2; collision mesh filename=./link_2.0.STL
- added link link_3; collision mesh filename=./link_3.0.STL
- added link link_4; collision mesh filename=./link_0.0.STL
- added link link_5; collision mesh filename=./link_1.0.STL
- added link link_6; collision mesh filename=./link_2.0.STL
- added link link_7; collision mesh filename=./link_3.0.STL
- added link link_8; collision mesh filename=./link_0.0.STL
- added link link_9; collision mesh filename=./link_1.0.STL
- added link mid_tip_tactile; collision mesh filename=./fingertip_V2_fixed2.STL scale=0.001 0.001 0.001
- added link ring_tip_tactile; collision mesh filename=./fingertip_V2_fixed2.STL scale=0.001 0.001 0.001
- added link thumb_tip_tactile; collision mesh filename=./fingertip_V2_fixed2.STL scale=0.001 0.001 0.001
- link palm_link: mass 0.4154 -> None; geometry collision mesh filename=./base_link.STL
Joints:
- removed joint joint_0.0
- removed joint joint_1.0
- removed joint joint_10.0
- removed joint joint_11.0
- removed joint joint_11.0_tip
- removed joint joint_12.0
- removed joint joint_13.0
- removed joint joint_14.0
- removed joint joint_15.0
- removed joint joint_15.0_tip
- removed joint joint_2.0
- removed joint joint_3.0
- removed joint joint_3.0_tip
- removed joint joint_4.0
- removed joint joint_5.0
- removed joint joint_6.0
- removed joint joint_7.0
- removed joint joint_7.0_tip
- removed joint joint_8.0
- removed joint joint_9.0
- added joint joint_0: type revolute, parent palm_link, child link_0, origin xyz=0 0.0435 -0.001542 rpy=-0.08726646255 0 0, axis 0 0 1, limit lower=-0.47 upper=0.47 effort=15 velocity=7
- added joint joint_1: type revolute, parent link_0, child link_1, origin xyz=0 0 0.0164, axis 0 1 0, limit lower=-0.196 upper=1.61 effort=15 velocity=7
- added joint joint_10: type revolute, parent link_9, child link_10, origin xyz=0 0 0.054, axis 0 1 0, limit lower=-0.174 upper=1.709 effort=15 velocity=7
- added joint joint_11: type revolute, parent link_10, child link_11, origin xyz=0 0 0.0384, axis 0 1 0, limit lower=-0.227 upper=1.618 effort=15 velocity=7
- added joint joint_12: type revolute, parent palm_link, child link_12, origin xyz=-0.0182 0.019333 -0.045987 rpy=0 -1.65806278845 -1.5707963259, axis -1 0 0, limit lower=0.263 upper=1.396 effort=15 velocity=7
- added joint joint_13: type revolute, parent link_12, child link_13, origin xyz=-0.027 0.005 0.0399, axis 0 0 1, limit lower=-0.105 upper=1.163 effort=15 velocity=7
- added joint joint_14: type revolute, parent link_13, child link_14, origin xyz=0 0 0.0177, axis 0 1 0, limit lower=-0.189 upper=1.644 effort=15 velocity=7
- added joint joint_15: type revolute, parent link_14, child link_15, origin xyz=0 0 0.0514, axis 0 1 0, limit lower=-0.162 upper=1.719 effort=15 velocity=7
- added joint joint_2: type revolute, parent link_1, child link_2, origin xyz=0 0 0.054, axis 0 1 0, limit lower=-0.174 upper=1.709 effort=15 velocity=7
- added joint joint_3: type revolute, parent link_2, child link_3, origin xyz=0 0 0.0384, axis 0 1 0, limit lower=-0.227 upper=1.618 effort=15 velocity=7
- added joint joint_4: type revolute, parent palm_link, child link_4, origin xyz=0 0 0.0007 rpy=0.0 0 0, axis 0 0 1, limit lower=-0.47 upper=0.47 effort=15 velocity=7
- added joint joint_5: type revolute, parent link_4, child link_5, origin xyz=0 0 0.0164, axis 0 1 0, limit lower=-0.196 upper=1.61 effort=15 velocity=7
- added joint joint_6: type revolute, parent link_5, child link_6, origin xyz=0 0 0.054, axis 0 1 0, limit lower=-0.174 upper=1.709 effort=15 velocity=7
- added joint joint_7: type revolute, parent link_6, child link_7, origin xyz=0 0 0.0384, axis 0 1 0, limit lower=-0.227 upper=1.618 effort=15 velocity=7
- added joint joint_8: type revolute, parent palm_link, child link_8, origin xyz=0 -0.0435 -0.001542 rpy=0.08726646255 0 0, axis 0 0 1, limit lower=-0.47 upper=0.47 effort=15 velocity=7
- added joint joint_9: type revolute, parent link_8, child link_9, origin xyz=0 0 0.0164, axis 0 1 0, limit lower=-0.196 upper=1.61 effort=15 velocity=7
- added joint joint_index_tip_tactile: type fixed, parent link_3, child index_tip_tactile, origin xyz=0.002 0 0.0157 rpy=0 0 0
- added joint joint_mid_tip_tactile: type fixed, parent link_7, child mid_tip_tactile, origin xyz=0.002 0 0.0157 rpy=0 0 0
- added joint joint_ring_tip_tactile: type fixed, parent link_11, child ring_tip_tactile, origin xyz=0.002 0 0.0157 rpy=0 0 0
- added joint joint_thumb_tip_tactile: type fixed, parent link_15, child thumb_tip_tactile, origin xyz=0.002 0 0.0313 rpy=0 0 0
